File: KiCad/YieldGuard.kicad_pcb (KiCad board)
At the start: 2 copper layers, 50 x 40 mm, 4 parts, among them J1 Conn_01x04_Socket, U1 ESP32_C3_Super_Mini, U2 HX711

Commit message: kicad fixes
Parts:
- moved G*** 1.95 mm to (114.3, 54.4)
Connections:
- U1 pad 1: /5V -> unconnected-(U1-5V-Pad1)
- U1 pad 3: unconnected-(U1-3.3V-Pad3) -> /PWR
- U2 pad 7: /5V -> /PWR
Routing:
- net /PWR: track 0.00 -> 71.0 mm
- net /5V: track 61.7 -> 0.00 mm
