File: KiCad/YieldGuard.kicad_sch (KiCad schematic)
At the start: 3 parts, among them J1 Conn_01x04_Socket, U1 ESP32-DEVKITC, U2 HX711

Commit message: Bit changes in PCB and Schematic and Completed BoM
Parts:
- removed U1: ESP32-DEVKITC, KiCad:MODULE_ESP32-DEVKITC, symbol ESP32-DEVKITC:ESP32-DEVKITC
- added U1: ESP32_C3_Super_Mini, KiCad:ESP32-C3_SuperMini, symbol ESP32-C3-SuperMini:ESP32_C2_Super_Mini
Connections:
- net 5V: now also U1.1 (5V)
- net CLOCK: now also U1.9 (GPIO5)
- net DATA: now also U1.4 (GPIO4)
- net GND: now also U1.2 (GND)
- no-connect marks 36 -> 14
Other:
- note added: "ESP32 C3 SuperMini"
- note removed: "ESP32 DevKitC V4"
- moved on the sheet: J1, U2

Commit message: kicad fixes
Connections:
- net PWR: now reaches U1.3 (3.3V)
- net PWR: now also U2.7 (VDD)
- net 5V: no longer names the net of U1.1 (5V)
- net 5V: no longer U2.7 (VDD)
Changed lines of the file:
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@@
-	)
-	(no_connect
-		(at 60.96 40.64)
 	)
 	(no_connect
@@
 	)
 	(no_connect
+		(at 62.23 35.56)
+	)
+	(no_connect
 		(at 30.48 50.8)
 	)
@@
 	(wire
 		(pts
+			(xy 127 34.29) (xy 128.27 34.29)
+		)
+		(stroke
+			(width 0)
+			(type default)
+		)
+	)
+	(wire
+		(pts
 			(xy 60.96 45.72) (xy 66.04 45.72)
 		)
@@
 	(wire
 		(pts
+			(xy 60.96 40.64) (xy 62.23 40.64)
+		)
+		(stroke
+			(width 0)
+			(type default)
+		)
+	)
+	(wire
+		(pts
 			(xy 68.58 93.98) (xy 85.09 93.98)
 		)
@@
 			(width 0)
 			(type default)
+		)
+	)
+	(label "PWR"
+		(at 128.27 34.29 0)
+		(effects
+			(font
+				(size 1.27 1.27)
+			)
+			(justify left bottom)
 		)
 	)
@@
 		)
 	)
+	(label "PWR"
+		(at 62.23 40.64 0)
+		(effects
+			(font
+				(size 1.27 1.27)
+			)
+			(justify left bottom)
+		)
+	)
 	(label "WHITE_WIRE"
 		(at 86.36 44.45 0)
@@
 		)
 	)
-	(label "5V"
-		(at 62.23 35.56 0)
-		(effects
-			(font
-				(size 1.27 1.27)
-			)
-			(justify left bottom)
-		)
-	)
 	(label "CLOCK"
 		(at 27.94 38.1 180)
@@
 		(effects
 			(font
-				(size 1.27 1.27)
-			)
-			(justify left bottom)
-		)
-	)
-	(label "5V"
-		(at 127 34.29 0)
-		(effects
-			(font
